Commit message: [config]: S54参数对齐实机

File: src/omni_gs_playground/assets/robots/kuavo/biped_s54/urdf/biped_s54.urdf (robot description, URDF)
Before this commit: robot biped_s54, 35 links, 34 joints
Links:
- removed link camera_base
- removed link head_rader
- added link dummy_link
- added link head_camera_base, mass 0.0; visual mesh filename=package://kuavo_assets/models/biped_s54/meshes/head_camera_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
- added link head_camera_depth, mass 0.0000785398163397463; visual mesh filename=package://kuavo_assets/models/biped_s54/meshes/head_camera_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
- added link head_radar, mass 0.0; visual mesh filename=package://kuavo_assets/models/biped_s54/meshes/head_radar.S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
- added link l_foot_heel; collision sphere radius=0.005
- added link l_foot_toe; collision sphere radius=0.005
- added link ll_foot_heel; collision sphere radius=0.005
- added link ll_foot_toe; collision sphere radius=0.005
- added link lr_foot_heel; collision sphere radius=0.005
- added link lr_foot_toe; collision sphere radius=0.005
- added link r_foot_heel; collision sphere radius=0.005
- added link r_foot_toe; collision sphere radius=0.005
- added link rl_foot_heel; collision sphere radius=0.005
- added link rl_foot_toe; collision sphere radius=0.005
- added link rr_foot_heel; collision sphere radius=0.005
- added link rr_foot_toe; collision sphere radius=0.005
- added link waist_camera_base, mass 0.13300000; visual mesh filename=package://kuavo_assets/models/biped_s54/meshes/waist_camera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
- link base_link: geometry collision cylinder length=0.24 radius=0.06; collision cylinder length=0.24 radius=0.06
- link leg_l1_link: geometry visual mesh filename=package://kuavo_assets/models/biped_s54/meshes/l_leg_roll.S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
- link leg_l2_link: geometry visual mesh filename=package://kuavo_assets/models/biped_s54/meshes/l_leg_yaw.STL
- link leg_l3_link: geometry collision capsule length=0.25 radius=0.065; collision cylinder length=0.04 radius=0.06
- link leg_l4_link: geometry collision capsule length=0.3 radius=0.05; visual mesh filename=package://kuavo_assets/models/biped_s54/meshes/l_knee.STL
- link leg_l5_link: geometry visual mesh filename=package://kuavo_assets/models/biped_s54/meshes/l_foot_pitch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
- link leg_l6_link: geometry collision box size=0.042 0.096 0.0108; collision box size=0.09 0.1 0.0108
- link leg_r1_link: geometry visual mesh filename=package://kuavo_assets/models/biped_s54/meshes/r_leg_roll.S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
- link leg_r2_link: geometry visual mesh filename=package://kuavo_assets/models/biped_s54/meshes/r_leg_yaw.STL
- link leg_r3_link: geometry collision capsule length=0.25 radius=0.065; collision cylinder length=0.04 radius=0.06
- link leg_r4_link: geometry collision capsule length=0.3 radius=0.05; visual mesh filename=package://kuavo_assets/models/biped_s54/meshes/r_knee.STL
- link leg_r5_link: geometry visual mesh filename=package://kuavo_assets/models/biped_s54/meshes/r_foot_pitch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
- link leg_r6_link: geometry collision box size=0.042 0.096 0.0108; collision box size=0.09 0.1 0.0108
- link waist_camera: mass 0.13300 -> 0.0000785398163397463; geometry visual mesh filename=package://kuavo_assets/models/biped_s54/meshes/waist_camera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
- link waist_yaw_link: mass 20.23838 -> 20.50328; geometry collision capsule length=0.06 radius=0.13; collision capsule length=0.12 radius=0.13
- link zarm_l1_link: geometry collision capsule length=0.04 radius=0.05; visual mesh filename=package://kuavo_assets/models/biped_s54/meshes/l_arm_pitch.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
- link zarm_l2_link: geometry visual mesh filename=package://kuavo_assets/models/biped_s54/meshes/l_arm_roll.S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
- link zarm_l3_link: geometry collision capsule length=0.14 radius=0.045; visual mesh filename=package://kuavo_assets/models/biped_s54/meshes/l_arm_yaw.STL
- link zarm_l4_link: geometry collision capsule length=0.18 radius=0.045; visual mesh filename=package://kuavo_assets/models/biped_s54/meshes/l_forearm.STL
- link zarm_l5_link: geometry visual mesh filename=package://kuavo_assets/models/biped_s54/meshes/l_hand_yaw.S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
- link zarm_l6_link: geometry visual mesh filename=package://kuavo_assets/models/biped_s54/meshes/l_hand_roll.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
- link zarm_l7_link: geometry collision box size=0.08 0.05 0.16; collision cylinder length=0.08 radius=0.01
- link zarm_r1_link: geometry collision capsule length=0.04 radius=0.05; visual mesh filename=package://kuavo_assets/models/biped_s54/meshes/r_arm_pitch.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
- link zarm_r2_link: geometry visual mesh filename=package://kuavo_assets/models/biped_s54/meshes/r_arm_roll.S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
- link zarm_r3_link: geometry collision capsule length=0.14 radius=0.045; visual mesh filename=package://kuavo_assets/models/biped_s54/meshes/r_arm_yaw.STL
- link zarm_r4_link: geometry collision capsule length=0.18 radius=0.045; visual mesh filename=package://kuavo_assets/models/biped_s54/meshes/r_forearm.STL
- link zarm_r5_link: geometry visual mesh filename=package://kuavo_assets/models/biped_s54/meshes/r_hand_yaw.S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
- link zarm_r6_link: geometry visual mesh filename=package://kuavo_assets/models/biped_s54/meshes/r_hand_roll.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
- link zarm_r7_link: geometry collision box size=0.08 0.05 0.16; collision cylinder length=0.08 radius=0.01
- link zhead_1_link: geometry visual mesh filename=package://kuavo_assets/models/biped_s54/meshes/head_yaw.STL
- link zhead_2_link: geometry collision sphere radius=0.1; visual mesh filename=package://kuavo_assets/models/biped_s54/meshes/head_pitch.S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
Joints:
- removed joint camera_base
- removed joint head_rader_joint
- removed joint waist_camera
- added joint dummy_to_base_link: type fixed, parent dummy_link, child base_link, origin xyz=0 0 0 rpy=0 0 0
- added joint head_camera_base_joint: type fixed, parent zhead_2_link, child head_camera_base, origin xyz=0.099619 0 0.032844 rpy=0 0.3406 0, axis 0 0 0
- added joint head_camera_depth_joint: type fixed, parent head_camera_base, child head_camera_depth, origin xyz=0.011715 0.0475 0.014312 rpy=0 0 0, axis 0 0 0
- added joint head_radar_joint: type fixed, parent zhead_1_link, child head_radar, origin xyz=0 0 -0.078453 rpy=0 0 0, axis 0 0 0
- added joint l_foot_heel_joint: type fixed, parent leg_l6_link, child l_foot_heel, origin xyz=-0.073164 0.0 -0.0595 rpy=0 0 0
- added joint l_foot_toe_joint: type fixed, parent leg_l6_link, child l_foot_toe, origin xyz=0.17084 0.0 -0.0595 rpy=0 0 0
- added joint ll_foot_heel_joint: type fixed, parent leg_l6_link, child ll_foot_heel, origin xyz=-0.073164 0.05 -0.0595 rpy=0 0 0
- added joint ll_foot_toe_joint: type fixed, parent leg_l6_link, child ll_foot_toe, origin xyz=0.17084 0.05 -0.0595 rpy=0 0 0
- added joint lr_foot_heel_joint: type fixed, parent leg_l6_link, child lr_foot_heel, origin xyz=-0.073164 -0.05 -0.0595 rpy=0 0 0
- added joint lr_foot_toe_joint: type fixed, parent leg_l6_link, child lr_foot_toe, origin xyz=0.17084 -0.05 -0.0595 rpy=0 0 0
- added joint r_foot_heel_joint: type fixed, parent leg_r6_link, child r_foot_heel, origin xyz=-0.073164 0.0 -0.0595 rpy=0 0 0
- added joint r_foot_toe_joint: type fixed, parent leg_r6_link, child r_foot_toe, origin xyz=0.17084 0.0 -0.0595 rpy=0 0 0
- added joint rl_foot_heel_joint: type fixed, parent leg_r6_link, child rl_foot_heel, origin xyz=-0.073164 0.05 -0.0595 rpy=0 0 0
- added joint rl_foot_toe_joint: type fixed, parent leg_r6_link, child rl_foot_toe, origin xyz=0.17084 0.05 -0.0595 rpy=0 0 0
- added joint rr_foot_heel_joint: type fixed, parent leg_r6_link, child rr_foot_heel, origin xyz=-0.073164 -0.05 -0.0595 rpy=0 0 0
- added joint rr_foot_toe_joint: type fixed, parent leg_r6_link, child rr_foot_toe, origin xyz=0.17084 -0.05 -0.0595 rpy=0 0 0
- added joint waist_camera_base_joint: type fixed, parent waist_yaw_link, child waist_camera_base, origin xyz=0.0787 0 -0.028149 rpy=0 0.59341 0, axis 0 0 0
- added joint waist_camera_joint: type fixed, parent waist_camera_base, child waist_camera, origin xyz=0.011715 0.0475 0.014312 rpy=0 0 0, axis 0 0 0
- joint leg_l6_joint: limit lower=-0.261799387799149 upper=0.261799387799149 effort=30.0 velocity=17.8 -> lower=-0.261799387799149 upper=0.261799387799149 effort=68.4 velocity=17.8
- joint leg_r6_joint: limit lower=-0.261799387799149 upper=0.261799387799149 effort=30.0 velocity=17.8 -> lower=-0.261799387799149 upper=0.261799387799149 effort=68.4 velocity=17.8
- joint zhead_1_joint: type fixed -> revolute
- joint zhead_2_joint: type fixed -> revolute
